Commit message: cv.py quasi completo , da controllare i vari if nel passaggio nello stato sleep e per fsm.py bisogna ricontrollare lo stato sleep, launch file modificato

File: urdf/robot.xacro (robot description, xacro)
@@ -154,11 +154,11 @@
     </visual>
    </link>
-   <joint name="joint_neck" type="revolute">
+   <joint name="joint_neck" type="fixed">
     <axis xyz="0 0 1"/>
     <origin rpy="0 0 0" xyz="0.15 0 0.075"/>
     <child link="link_neck"/>
     <parent link="link_chassis"/>
-    <limit effort="10000" lower="-0.7" upper="0.7" velocity="1000"/>
-    <joint_properties damping="1.0" friction="1.0"/>
+    <!--<limit effort="10000" lower="-0.7" upper="0.7" velocity="1000"/>
+    <joint_properties damping="1.0" friction="1.0"/> -->
    </joint>
    <joint name="joint_head" type="fixed">

Commit message: fsm.py completed but moving of the neck is not working, cv.py and launch file are ok!

File: urdf/robot.xacro (robot description, xacro)
@@ -212,4 +212,15 @@
 	    <child link="camera_link"/>
 	 </joint>
-<!--  Transmission to control the rotation of the neck -->
+<!--  Transmission to control the rotation of the neck
+<transmission name="head_joint_trans">
+  <type>transmission_interface/SimpleTransmission</type>
+  <joint name="head_joint">
+    <hardwareInterface>hardware_interface/EffortJointInterface</hardwareInterface>
+  </joint>
+  <actuator name="motor1">
+    <hardwareInterface>hardware_interface/EffortJointInterface</hardwareInterface>
+    <mechanicalInterface>1</mechanicalInterface>
+  </actuator>
+</transmission>
+-->
 </robot>
